File: beeping-easter-egg.kicad_pcb (KiCad board)
At the start: 2 copper layers, 84 x 38 mm, 19 parts, among them Q1 AO3401A, Q2 AO3401A, SW1 YUEN FUNG ST-0-102-A01-T000-LF, U1 TLC555CDR

Commit message: Add another mounting hole for cover plate. Move Q1 and R3 to make room for new mounting hole.
Parts:
- added REF**: MountingHole_3.2mm_M3, MountingHole:MountingHole_3.2mm_M3, F.Cu at (184.0, 90.0)
- added REF**: MountingHole_3.2mm_M3, MountingHole:MountingHole_3.2mm_M3, F.Cu at (138.0, 90.0)
- moved Q1 30.7 mm to (163.2, 108.3)
- moved R3 30.7 mm to (160.2, 110.1)
Routing:
- net VCC: track 28.2 -> 51.3 mm
- net Net-(Q1-D): track 15.3 -> 19.2 mm

Commit message: Separate cover into separate kicad_pcb file.
Parts:
- removed the REF** at (206.0, 93.3)
- removed the REF** at (201.4, 114.0)
- removed the REF** at (210.9, 101.7)
- removed the REF** at (184.0, 90.0)
Routing:
- removed copper zone on B.Cu, net (none)
- removed copper zone on F.Cu, net (none)
Other:
- board size 84 x 38 mm -> 38 x 38 mm

Commit message: Update title
Other:
- board text added: "github.com/DougTomanio /beeping-easter-egg Rev B"
- board text removed: "Beeping Easter Egg Rev B"
Changed lines of the file:
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@@
 		(layer "Edge.Cuts")
 	)
-	(gr_text "Beeping Easter Egg\nRev B"
-		(at 150 111.5 0)
+	(gr_text "github.com/DougTomanio\n/beeping-easter-egg\nRev B"
+		(at 150 110.5 0)
 		(layer "B.Cu")
 		(effects
